File: hw/scr_precharge_single_REV_B/scr_precharge.sch (EAGLE design)
At the start: 49 parts, among them IC1 LM311D, Q1 NTR5198NL, Q2 NTR5198NL, T1 78601, T2 78601, U1 ATTINY85DIL8, X1 +5V, X2 AC IN, X3 PRECHG, X4 RUN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

Commit message: added BOMs
Parts:
- Q1, Q2: value NTR5198NL -> SSM3K341R.LF
Changed lines of the file:
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@@
 <part name="C6" library="resistor" deviceset="C-EU" device="C0805" value="1u"/>
 <part name="D5" library="diode" deviceset="SMAZ12-TP" device=""/>
-<part name="Q1" library="SparkFun-DiscreteSemi" deviceset="MOSFET-NCH" device="-AO3404A" value="NTR5198NL"/>
+<part name="Q1" library="SparkFun-DiscreteSemi" deviceset="MOSFET-NCH" device="-AO3404A" value="SSM3K341R.LF"/>
 <part name="GND11" library="supply1" deviceset="GND" device=""/>
 <part name="D4" library="diode" deviceset="1N4148" device="MICROMELF" value="1N4148MICROMELF"/>
@@
 <part name="C8" library="resistor" deviceset="C-EU" device="C0805" value="1u"/>
 <part name="D7" library="diode" deviceset="SMAZ12-TP" device=""/>
-<part name="Q2" library="SparkFun-DiscreteSemi" deviceset="MOSFET-NCH" device="-AO3404A" value="NTR5198NL"/>
+<part name="Q2" library="SparkFun-DiscreteSemi" deviceset="MOSFET-NCH" device="-AO3404A" value="SSM3K341R.LF"/>
 <part name="GND12" library="supply1" deviceset="GND" device=""/>
 <part name="D6" library="diode" deviceset="1N4148" device="MICROMELF" value="1N4148MICROMELF"/>
